File: Main Board.brd (EAGLE design)
At the start: 90 x 90 mm, 106 parts, among them Q1 NVMFS5C604NLAFT1G, Q10 BSS123N_H6327, Q2 NVMFS5C604NLAFT1G, Q3 NVMFS5C604NLAFT1G, Q4 NVMFS5C604NLAFT1G, Q5 NVMFS5C604NLAFT1G, Q6 NVMFS5C604NLAFT1G, Q7 FDBL86361-F085, Q8 FDBL86361-F085, Q9 2N7002BK, U1 A4964EVTR-T, U2 LM74700-Q1MKX-1_NOPB, U4 STM8AF62X3

Commit message: Files Updated 5-21
Parts:
- added C8: 0.1uF, 25V, CGA3E2X7R1E104K080AA:CAPC1608X90N
- C60: value .1uF, 25V -> 0.1uF, 25V
- U4: value STM8AF62X3 -> STM8AF62X6T; device STM8AF6223PDU:TSSOP20 -> STM8AF6266T:LQFP-32
- moved U$2 66.1 mm to (113.0, 43.2)
- moved U$1 66.0 mm to (113.0, 47.0)
- moved U$4 64.8 mm to (108.0, 43.2)
- moved U$3 64.8 mm to (108.0, 47.0)
- moved JP1 7.90 mm to (78.6, 64.1), turned to 90 degrees
- moved C62 5.71 mm to (69.2, 69.8), turned to 90 degrees
- moved U4 2.90 mm to (69.6, 62.4)
- moved JP2 2.84 mm to (85.1, 57.1)
- moved C4 1.80 mm to (8.89, 54.6)
- moved JP3 1.27 mm to (86.5, 49.7)
Connections:
- new net N$12: U4.3
- new net N$13: U4.15
- new net N$15: U4.13
- new net N$20: U4.12
- new net N$21: U4.11
- new net N$22: U4.18
- new net N$23: U4.20
- new net N$25: U4.25
- new net N$26: U4.27
- new net N$27: U4.28
- new net N$28: U4.29
- new net N$29: U4.32
- new net N$30: U4.8
- new net N$31: U1.13
- new net N$32: U1.14
- new net N$6: C8.2, U4.6, U4.7
- new net N$9: U4.2
- net ANALOGIN: now also U4.14; no longer U4.19
- net GND: now also C8.1, U4.10, U4.4; no longer U4.7
- net LINUARTRXD: now also U4.31; no longer U4.3
- net LINUARTTXD: now also U4.30; no longer U4.2
- net NRST: now also U4.1; no longer U4.4
- net PWMIN: now also U4.19; no longer U4.13
- net SPI_MISO: now also U4.24; no longer U4.17
- net SPI_MOSI: now also U4.23; no longer U4.16
- net SPI_NSS: now also U4.17; no longer U4.14
- net SPI_SCK: now also U4.22; no longer U4.15
- net SWIM: now also U4.26; no longer U4.18
- net TEMPSENSOR: now also U4.16; no longer U4.20
- net VCAP: now also U4.5; no longer U4.8
- net WDOG: now also U4.21; no longer U4.10
Routing:
- net ANALOGIN: track 13.4 -> 27.6 mm, vias 4 -> 5
- net GND: track 79.2 -> 89.4 mm, vias 64 -> 68
- net NRST: track 43.8 -> 50.5 mm
- net TEMPSENSOR: track 7.55 -> 13.3 mm
- net SWIM: track 14.1 -> 8.63 mm, vias 2 -> 0
- net SPI_MISO: track 28.0 -> 32.7 mm
- net N$6: track 0.00 -> 4.11 mm
- net VCC: track 16.8 -> 20.6 mm
- net SPI_MOSI: track 26.6 -> 29.2 mm
- net SPI_SCK: track 26.9 -> 29.5 mm
- net WDOG: track 32.2 -> 29.6 mm
- net SPI_NSS: track 27.2 -> 29.2 mm
- net PWMIN: track 5.26 -> 6.20 mm
- net N$1: track 84.2 -> 83.6 mm
- net ANALOG_CMD: track 10.2 -> 10.7 mm
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Other:
- board text added: "+24V"
- board text added: "A"
- board text added: "D"
- board text added: "GND"
- board text added: "P"
- board text added: "R"
- board text added: "T"
- board text removed: "1000 mil"
- board text removed: "2in^2"
- board text removed: "5in^2"
