File: Main Board.sch (EAGLE design)
At the start: 106 parts, among them Q1 NVMFS5C604NLAFT1G, Q10 BSS123N_H6327, Q2 NVMFS5C604NLAFT1G, Q3 NVMFS5C604NLAFT1G, Q4 NVMFS5C604NLAFT1G, Q5 NVMFS5C604NLAFT1G, Q6 NVMFS5C604NLAFT1G, Q7 FDBL86361-F085, Q8 FDBL86361-F085, Q9 2N7002BK, U1 A4964EVTR-T, U2 LM74700-Q1MKX-1_NOPB, U4 STM8AF62X3

Commit message: Files Updated 5-21
Parts:
- added C8: 0.1uF, 25V, CGA3E2X7R1E104K080AA:CGA3E2X7R1E104K080AA
- added U$10, U$11, U$12, U$13, U$14, U$15, U$16, U$17, U$18, U$19, U$20, U$5, U$6, U$7, U$8, U$9: NC, BLDCBOMv4:NC
- C60: value .1uF, 25V -> 0.1uF, 25V
- U4: value STM8AF62X3 -> STM8AF62X6T; device STM8AF6223PDU:STM8AF62X3 -> STM8AF6266T:STM8AF62X6T
Connections:
- new net N$12: U$8.D, U4A.PA2/OSCOUT
- new net N$13: U$11.D, U4A.PB1
- new net N$15: U$9.D, U4A.PB3
- new net N$20: U$10.D, U4A.PB4
- new net N$21: U$12.D, U4A.PB5
- new net N$22: U$13.D, U4A.PC1
- new net N$23: U$20.D, U4A.PC3
- new net N$25: U$14.D, U4A.PD0
- new net N$26: U$15.D, U4A.PD2
- new net N$27: U$16.D, U4A.PD3
- new net N$28: U$17.D, U4A.PD4
- new net N$29: U$18.D, U4A.PD7
- new net N$30: U$19.D, U4A.PF4
- new net N$31: U$5.D, U1.LRX
- new net N$32: U$6.D, U1.LTX
- new net N$6: C8.2, U4B.VDD, U4B.VDDIO_1
- new net N$9: U$7.D, U4A.PA1/OSCIN
- net ANALOGIN: now also U4A.PB2; no longer U4.PD2/AIN3[TIM5_CH3]
- net GND: now also C8.1, U4B.VSS, U4B.VSSA; no longer U4.VSS
- net LINUARTRXD: now also U4A.PD6; no longer U4.PD6
- net LINUARTTXD: now also U4A.PD5; no longer U4.PD5
- net NRST: now also U4A.NRST; no longer U4.NRST
- net PWMIN: now also U4A.PC2; no longer U4.PC3
- net SPI_MISO: now also U4A.PC7; no longer U4.PC7
- net SPI_MOSI: now also U4A.PC6; no longer U4.PC6
- net SPI_NSS: now also U4A.PE5; no longer U4.PC4
- net SPI_SCK: now also U4A.PC5; no longer U4.PC5
- net SWIM: now also U4A.PD1; no longer U4.PD1
- net TEMPSENSOR: now also U4A.PB0; no longer U4.PD3/AIN4/TIM5_CH2/ADC_ETR
- net VCAP: now also U4B.VCAP; no longer U4.VCAP
- net VDD: now also U4B.VDDA; no longer U4.VDD
- net WDOG: now also U4A.PC4; no longer U4.PA3
Other:
- note added: "VCAP Pg 62 min value of 470 nF max value of 3300 nF"
- note removed: "VCAP Pg 56 min value of 470 nF max value of 3300 nF"
- moved on the sheet: C60, C61, C62, JP2
